File: hardware/laser_sensor/laser_sensor.brd (EAGLE design)
At the start: 28.6 x 23.5 mm, 11 parts, among them IC1 NE555D, J1 B4B-XH-A(LF)(SN)

Commit message: laser sensor gerber updated
Other:
- board text added: "DO NOT TOUCH ===>"
- board text added: "v0.1-alpha"
- board text added: "λ:"
- board text removed: "v1.0"
Changed lines of the file:
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@@
 <hole x="3.81" y="3.81" drill="2.9972"/>
 <hole x="24.765" y="19.685" drill="2.9972"/>
-<text x="8.255" y="8.255" size="1.778" layer="51">v1.0</text>
+<text x="1.905" y="7.62" size="1.778" layer="25">v0.1-alpha</text>
+<text x="14.605" y="12.7" size="1.778" layer="26" rot="MR0">DO NOT
+TOUCH
+===&gt;</text>
+<text x="23.495" y="8.89" size="3.175" layer="26" rot="MR0">λ:</text>
+<rectangle x1="8.255" y1="8.89" x2="20.32" y2="12.065" layer="26"/>
 </plain>
 <attributes>
@@
 </drawing>
 <compatibility>
+<note version="6.3" minversion="6.2.2" severity="warning">
+Since Version 6.2.2 text objects can contain more than one line,
+which will not be processed correctly with this version.
+</note>
 <note version="8.2" severity="warning">
 Since Version 8.2, EAGLE supports online libraries. The ids
