File: hardware/laser_sensor/laser_sensor.sch (EAGLE design)
At the start: 8 parts, among them J1 B4B-XH-A(LF)(SN), Q1 BC817-16LT1SMD

Commit message: updated pdf added for sensor
Other:
- note added: "v1.0"
- note removed: "v0.1_α"
Changed lines of the file:
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@@
 <?xml version="1.0" encoding="utf-8"?>
 <!DOCTYPE eagle SYSTEM "eagle.dtd">
-<eagle version="9.2.2">
+<eagle version="9.1.3">
 <drawing>
 <settings>
@@
 <sheet>
 <plain>
-<text x="246.38" y="5.08" size="2.54" layer="94">v0.1_α</text>
+<text x="246.38" y="5.08" size="2.54" layer="94">v1.0</text>
 </plain>
 <instances>

Commit message: changed some transistors
Parts:
- removed Q1: BC817-16LT1SMD, transistor-npn:BC817-16LT1SMD
- removed R2: 100k, rcl:R-US_R0603
- removed R3: 10k, rcl:R-US_R0603
- added T1: (no value), transistor:MUN2214T1-NPN_DRIVER-SC59-BEC
Connections:
- removed net N$3: Q1.B, R2.1, R3.2
- net GND: now also T1.E; no longer Q1.E, R2.2
- net LED: now also T1.B; no longer R3.1
- net N$2: now also T1.C; no longer Q1.C
Changed lines of the file:
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@@
 <part name="R1" library="rcl" library_urn="urn:adsk.eagle:library:334" deviceset="R-US_" device="R0603" package3d_urn="urn:adsk.eagle:package:23555/2" value="100k"/>
 <part name="GND1" library="supply1" library_urn="urn:adsk.eagle:library:371" deviceset="GND" device=""/>
-<part name="Q1" library="transistor-npn" library_urn="urn:adsk.eagle:library:398" deviceset="BC817*" device="SMD" package3d_urn="urn:adsk.eagle:package:28990/2" technology="-16LT1"/>
-<part name="R2" library="rcl" library_urn="urn:adsk.eagle:library:334" deviceset="R-US_" device="R0603" package3d_urn="urn:adsk.eagle:package:23555/2" value="100k"/>
-<part name="R3" library="rcl" library_urn="urn:adsk.eagle:library:334" deviceset="R-US_" device="R0603" package3d_urn="urn:adsk.eagle:package:23555/2" value="10k"/>
 <part name="R4" library="rcl" library_urn="urn:adsk.eagle:library:334" deviceset="R-US_" device="R0603" package3d_urn="urn:adsk.eagle:package:23555/2" value="560"/>
 <part name="P+2" library="supply1" library_urn="urn:adsk.eagle:library:371" deviceset="+5V" device=""/>
 <part name="GND2" library="supply1" library_urn="urn:adsk.eagle:library:371" deviceset="GND" device=""/>
+<part name="T1" library="transistor" library_urn="urn:adsk.eagle:library:402" deviceset="*-NPN_DRIVER-" device="SC59-BEC" package3d_urn="urn:adsk.eagle:package:29926/2" technology="MUN2214T1"/>
 </parts>
 <sheets>
@@
 <attribute name="VALUE" x="78.74" y="60.96" size="1.778" layer="96"/>
 </instance>
-<instance part="Q1" gate="G$1" x="160.02" y="81.28" smashed="yes">
-<attribute name="NAME" x="149.86" y="88.9" size="1.778" layer="95"/>
-<attribute name="VALUE" x="149.86" y="86.36" size="1.778" layer="96"/>
-</instance>
-<instance part="R2" gate="G$1" x="154.94" y="73.66" smashed="yes">
-<attribute name="NAME" x="151.13" y="75.1586" size="1.778" layer="95"/>
-<attribute name="VALUE" x="151.13" y="70.358" size="1.778" layer="96"/>
-</instance>
-<instance part="R3" gate="G$1" x="139.7" y="81.28" smashed="yes">
-<attribute name="NAME" x="135.89" y="82.7786" size="1.778" layer="95"/>
-<attribute name="VALUE" x="135.89" y="77.978" size="1.778" layer="96"/>
-</instance>
 <instance part="R4" gate="G$1" x="162.56" y="106.68" smashed="yes" rot="R90">
 <attribute name="NAME" x="161.0614" y="102.87" size="1.778" layer="95" rot="R90"/>
@@
 <attribute name="VALUE" x="160.02" y="60.96" size="1.778" layer="96"/>
 </instance>
+<instance part="T1" gate="G$1" x="160.02" y="81.28"/>
 </instances>
 <busses>
@@
 </segment>
 <segment>
-<pinref part="R2" gate="G$1" pin="2"/>
-<wire x1="160.02" y1="73.66" x2="162.56" y2="73.66" width="0.1524" layer="91"/>
-<pinref part="Q1" gate="G$1" pin="E"/>
-<wire x1="162.56" y1="73.66" x2="162.56" y2="76.2" width="0.1524" layer="91"/>
+<pinref part="T1" gate="G$1" pin="E"/>
 <pinref part="GND2" gate="1" pin="GND"/>
-<wire x1="162.56" y1="66.04" x2="162.56" y2="73.66" width="0.1524" layer="91"/>
-<junction x="162.56" y="73.66"/>
+<wire x1="162.56" y1="76.2" x2="162.56" y2="66.04" width="0.1524" layer="91"/>
 </segment>
 </net>
@@
 </segment>
 <segment>
-<pinref part="R3" gate="G$1" pin="1"/>
-<wire x1="134.62" y1="81.28" x2="129.54" y2="81.28" width="0.1524" layer="91"/>
 <label x="129.54" y="81.28" size="1.778" layer="95" rot="R180" xref="yes"/>
+<wire x1="129.54" y1="81.28" x2="152.4" y2="81.28" width="0.1524" layer="91"/>
+<pinref part="T1" gate="G$1" pin="B"/>
 </segment>
 </net>
@@
 <net name="N$2" class="0">
 <segment>
+<pinref part="T1" gate="G$1" pin="C"/>
 <pinref part="LED1" gate="G$1" pin="C"/>
-<pinref part="Q1" gate="G$1" pin="C"/>
-<wire x1="162.56" y1="91.44" x2="162.56" y2="86.36" width="0.1524" layer="91"/>
+<wire x1="162.56" y1="86.36" x2="162.56" y2="91.44" width="0.1524" layer="91"/>
 </segment>
 </net>
-<net name="N$3" class="0">
-<segment>
-<pinref part="Q1" gate="G$1" pin="B"/>
-<pinref part="R3" gate="G$1" pin="2"/>
-<wire x1="157.48" y1="81.28" x2="147.32" y2="81.28" width="0.1524" layer="91"/>
-<pinref part="R2" gate="G$1" pin="1"/>
-<wire x1="147.32" y1="81.28" x2="144.78" y2="81.28" width="0.1524" layer="91"/>
-<wire x1="149.86" y1="73.66" x2="147.32" y2="73.66" width="0.1524" layer="91"/>
-<wire x1="147.32" y1="73.66" x2="147.32" y2="81.28" width="0.1524" layer="91"/>
-<junction x="147.32" y="81.28"/>
-</segment>
-</net>
