File: hardware/speedometer/speedometer.sch (EAGLE design)
At the start: 139 parts, among them IC1 PIC32MX110F016B-I_SO, IC10 24LC024SN, IC11 MAX16054AZT+T, IC12 TPS63001DRCT, IC13 TPS63002DRCT, IC2 CSTCE8M00G55-R0, IC3 CSTCE12M0G15L99-R0, IC4 MCP2200-I_SO, IC6 PCF8574T, IC7 BQ24075RGTT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

Commit message: Most of the work is done. Fixing ground planes and power paths
Parts:
- removed R18: 100, rcl:R-US_R0805
- removed TP24: TPB1,27, testpad:TPB1,27
- C5, C9: device rcl:C-EUC0805 -> rcl:C-EUC0805K
- TP14: TP_SIGNAL_NAME TP_MCLR -> TP_!MCLR
Connections:
- removed net N$11: IC7.SYSOFF, R18.2, TP24.TP
- removed net N$16: IC6.P0, R17.1
- new net N$3: IC6.P3, R17.1
- net !MCLR: no longer TP14.TP
- net !SYSOFF: no longer R18.1
- net GND: now also IC7.SYSOFF
- net LASER_LEFT_CTL: now also IC6.P0; no longer IC6.P3
- net LEFT_STS: now also IC6.P2; no longer IC6.P1
- net N$42: now also TP14.TP
- net RIGHT_STS: now also IC6.P1; no longer IC6.P2
Other:
- moved on the sheet: LED5, R17

Commit message: Routing is done. Waiting a check from a Sandro
Parts:
- C1, C10, C2, C22, C23, C24, C3, C6, C7, C8, C9: device rcl:C-EUC0805K -> rcl:C-EUC0603K
- C12: device rcl:C-EUC0805 -> rcl:C-EUC0603K
Changed lines of the file:
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@@
 <setting verticaltext="up"/>
 </settings>
-<grid distance="0.1" unitdist="inch" unit="inch" style="lines" multiple="1" display="yes" altdistance="0.01" altunitdist="inch" altunit="inch"/>
+<grid distance="0.1" unitdist="inch" unit="inch" style="lines" multiple="1" display="no" altdistance="0.01" altunitdist="inch" altunit="inch"/>
 <layers>
 <layer number="1" name="Top" color="4" fill="1" visible="no" active="no"/>
@@
 <part name="GND22" library="supply1" library_urn="urn:adsk.eagle:library:371" deviceset="GND" device=""/>
 <part name="GND21" library="supply1" library_urn="urn:adsk.eagle:library:371" deviceset="GND" device=""/>
-<part name="C9" library="rcl" library_urn="urn:adsk.eagle:library:334" deviceset="C-EU" device="C0805K" package3d_urn="urn:adsk.eagle:package:23681/2" value="100n"/>
+<part name="C9" library="rcl" library_urn="urn:adsk.eagle:library:334" deviceset="C-EU" device="C0603K" package3d_urn="urn:adsk.eagle:package:23680/2" value="100n"/>
 <part name="+3V39" library="supply1" library_urn="urn:adsk.eagle:library:371" deviceset="+3V3" device=""/>
 <part name="SV2" library="con-lstb" library_urn="urn:adsk.eagle:library:162" deviceset="MA05-2" device="" package3d_urn="urn:adsk.eagle:package:8329/1"/>
@@
 <part name="+3V38" library="supply1" library_urn="urn:adsk.eagle:library:371" deviceset="+3V3" device=""/>
 <part name="R13" library="rcl" library_urn="urn:adsk.eagle:library:334" deviceset="R-US_" device="R0805" package3d_urn="urn:adsk.eagle:package:23553/2" value="10k"/>
-<part name="C8" library="rcl" library_urn="urn:adsk.eagle:library:334" deviceset="C-EU" device="C0805K" package3d_urn="urn:adsk.eagle:package:23681/2" value="100n"/>
+<part name="C8" library="rcl" library_urn="urn:adsk.eagle:library:334" deviceset="C-EU" device="C0603K" package3d_urn="urn:adsk.eagle:package:23680/2" value="100n"/>
 <part name="GND20" library="supply1" library_urn="urn:adsk.eagle:library:371" deviceset="GND" device=""/>
 <part name="SJ1" library="jumper" library_urn="urn:adsk.eagle:library:252" deviceset="SJ" device="" package3d_urn="urn:adsk.eagle:package:15471/1"/>
@@
 <part name="+3V313" library="supply1" library_urn="urn:adsk.eagle:library:371" deviceset="+3V3" device=""/>
 <part name="+3V310" library="supply1" library_urn="urn:adsk.eagle:library:371" deviceset="+3V3" device=""/>
-<part name="C10" library="rcl" library_urn="urn:adsk.eagle:library:334" deviceset="C-EU" device="C0805K" package3d_urn="urn:adsk.eagle:package:23681/2" value="100n"/>
+<part name="C10" library="rcl" library_urn="urn:adsk.eagle:library:334" deviceset="C-EU" device="C0603K" package3d_urn="urn:adsk.eagle:package:23680/2" value="100n"/>
 <part name="GND27" library="supply1" library_urn="urn:adsk.eagle:library:371" deviceset="GND" device=""/>
 <part name="FRAME5" library="frames" library_urn="urn:adsk.eagle:library:229" deviceset="A4L-LOC" device=""/>
@@
 <part name="J2" library="B2B-PH-SM4-TB(LF)(SN)" deviceset="B2B-PH-SM4-TB(LF)(SN)" device="" value="BAT"/>
 <part name="GND31" library="supply1" library_urn="urn:adsk.eagle:library:371" deviceset="GND" device=""/>
-<part name="C12" library="rcl" library_urn="urn:adsk.eagle:library:334" deviceset="C-EU" device="C0805" package3d_urn="urn:adsk.eagle:package:23617/2" value="100n"/>
+<part name="C12" library="rcl" library_urn="urn:adsk.eagle:library:334" deviceset="C-EU" device="C0603K" package3d_urn="urn:adsk.eagle:package:23680/2" value="100n"/>
 <part name="GND33" library="supply1" library_urn="urn:adsk.eagle:library:371" deviceset="GND" device=""/>
 <part name="LED7" library="led" library_urn="urn:adsk.eagle:library:259" deviceset="LED" device="3MM" package3d_urn="urn:adsk.eagle:package:15797/1"/>
@@
 <part name="+3V35" library="supply1" library_urn="urn:adsk.eagle:library:371" deviceset="+3V3" device=""/>
 <part name="+3V31" library="supply1" library_urn="urn:adsk.eagle:library:371" deviceset="+3V3" device=""/>
-<part name="C1" library="rcl" library_urn="urn:adsk.eagle:library:334" deviceset="C-EU" device="C0805K" package3d_urn="urn:adsk.eagle:package:23681/2" value="100n"/>
-<part name="C3" library="rcl" library_urn="urn:adsk.eagle:library:334" deviceset="C-EU" device="C0805K" package3d_urn="urn:adsk.eagle:package:23681/2" value="100n"/>
+<part name="C1" library="rcl" library_urn="urn:adsk.eagle:library:334" deviceset="C-EU" device="C0603K" package3d_urn="urn:adsk.eagle:package:23680/2" value="100n"/>
+<part name="C3" library="rcl" library_urn="urn:adsk.eagle:library:334" deviceset="C-EU" device="C0603K" package3d_urn="urn:adsk.eagle:package:23680/2" value="100n"/>
 <part name="GND8" library="supply1" library_urn="urn:adsk.eagle:library:371" deviceset="GND" device=""/>
 <part name="GND1" library="supply1" library_urn="urn:adsk.eagle:library:371" deviceset="GND" device=""/>
 <part name="R2" library="resistor" library_urn="urn:adsk.eagle:library:348" deviceset="R-US_" device="M0805" package3d_urn="urn:adsk.eagle:package:26079/1" value="1k"/>
 <part name="R1" library="resistor" library_urn="urn:adsk.eagle:library:348" deviceset="R-US_" device="M0805" package3d_urn="urn:adsk.eagle:package:26079/1" value="10k"/>
-<part name="C2" library="rcl" library_urn="urn:adsk.eagle:library:334" deviceset="C-EU" device="C0805K" package3d_urn="urn:adsk.eagle:package:23681/2" value="100n"/>
+<part name="C2" library="rcl" library_urn="urn:adsk.eagle:library:334" deviceset="C-EU" device="C0603K" package3d_urn="urn:adsk.eagle:package:23680/2" value="100n"/>
 <part name="+3V32" library="supply1" library_urn="urn:adsk.eagle:library:371" deviceset="+3V3" device=""/>
 <part name="GND3" library="supply1" library_urn="urn:adsk.eagle:library:371" deviceset="GND" device=""/>
@@
 <part name="GND13" library="supply1" library_urn="urn:adsk.eagle:library:371" deviceset="GND" device=""/>
 <part name="VDD2" library="supply1" library_urn="urn:adsk.eagle:library:371" deviceset="VDD" device=""/>
-<part name="C7" library="rcl" library_urn="urn:adsk.eagle:library:334" deviceset="C-EU" device="C0805K" package3d_urn="urn:adsk.eagle:package:23681/2" value="100n"/>
+<part name="C7" library="rcl" library_urn="urn:adsk.eagle:library:334" deviceset="C-EU" device="C0603K" package3d_urn="urn:adsk.eagle:package:23680/2" value="100n"/>
 <part name="GND17" library="supply1" library_urn="urn:adsk.eagle:library:371" deviceset="GND" device=""/>
 <part name="GND15" library="supply1" library_urn="urn:adsk.eagle:library:371" deviceset="GND" device=""/>
@@
 <part name="R6" library="rcl" library_urn="urn:adsk.eagle:library:334" deviceset="R-US_" device="R0805" package3d_urn="urn:adsk.eagle:package:23553/2" value="4k7"/>
 <part name="VDD3" library="supply1" library_urn="urn:adsk.eagle:library:371" deviceset="VDD" device=""/>
-<part name="C6" library="rcl" library_urn="urn:adsk.eagle:library:334" deviceset="C-EU" device="C0805K" package3d_urn="urn:adsk.eagle:package:23681/2" value="100n"/>
+<part name="C6" library="rcl" library_urn="urn:adsk.eagle:library:334" deviceset="C-EU" device="C0603K" package3d_urn="urn:adsk.eagle:package:23680/2" value="100n"/>
 <part name="GND12" library="supply1" library_urn="urn:adsk.eagle:library:371" deviceset="GND" device=""/>
 <part name="T1" library="transistor-neu-to92" library_urn="urn:adsk.eagle:library:397" deviceset="*-NPN-" device="SOT23-BEC" package3d_urn="urn:adsk.eagle:package:28748/2" technology="BC817-16"/>
@@
 <part name="GND53" library="supply1" library_urn="urn:adsk.eagle:library:371" deviceset="GND" device=""/>
 <part name="GND52" library="supply1" library_urn="urn:adsk.eagle:library:371" deviceset="GND" device=""/>
-<part name="C22" library="rcl" library_urn="urn:adsk.eagle:library:334" deviceset="C-EU" device="C0805K" package3d_urn="urn:adsk.eagle:package:23681/2" value="100n"/>
+<part name="C22" library="rcl" library_urn="urn:adsk.eagle:library:334" deviceset="C-EU" device="C0603K" package3d_urn="urn:adsk.eagle:package:23680/2" value="100n"/>
 <part name="+3V320" library="supply1" library_urn="urn:adsk.eagle:library:371" deviceset="+3V3" device=""/>
 <part name="GND51" library="supply1" library_urn="urn:adsk.eagle:library:371" deviceset="GND" device=""/>
@@
 <part name="VCC2" library="supply1" library_urn="urn:adsk.eagle:library:371" deviceset="VCCINT" device=""/>
 <part name="R36" library="rcl" library_urn="urn:adsk.eagle:library:334" deviceset="R-US_" device="R0805" package3d_urn="urn:adsk.eagle:package:23553/2" value="100"/>
-<part name="C23" library="rcl" library_urn="urn:adsk.eagle:library:334" deviceset="C-EU" device="C0805K" package3d_urn="urn:adsk.eagle:package:23681/2" value="100n"/>
+<part name="C23" library="rcl" library_urn="urn:adsk.eagle:library:334" deviceset="C-EU" device="C0603K" package3d_urn="urn:adsk.eagle:package:23680/2" value="100n"/>
 <part name="GND54" library="supply1" library_urn="urn:adsk.eagle:library:371" deviceset="GND" device=""/>
 <part name="GND57" library="supply1" library_urn="urn:adsk.eagle:library:371" deviceset="GND" device=""/>
@@
 <part name="VCC3" library="supply1" library_urn="urn:adsk.eagle:library:371" deviceset="VCCINT" device=""/>
 <part name="R37" library="rcl" library_urn="urn:adsk.eagle:library:334" deviceset="R-US_" device="M0805" package3d_urn="urn:adsk.eagle:package:23556/1" value="100"/>
-<part name="C24" library="rcl" library_urn="urn:adsk.eagle:library:334" deviceset="C-EU" device="C0805K" package3d_urn="urn:adsk.eagle:package:23681/2" value="100n"/>
+<part name="C24" library="rcl" library_urn="urn:adsk.eagle:library:334" deviceset="C-EU" device="C0603K" package3d_urn="urn:adsk.eagle:package:23680/2" value="100n"/>
 <part name="GND55" library="supply1" library_urn="urn:adsk.eagle:library:371" deviceset="GND" device=""/>
 <part name="GND58" library="supply1" library_urn="urn:adsk.eagle:library:371" deviceset="GND" device=""/>

Commit message: WIP
Parts:
- T1: value (none) -> BC817-16LT1SMD; device transistor-neu-to92:BC817-16-NPN-SOT23-BEC -> transistor-npn:BC817-16LT1SMD
- renumbered SV1 to ICSP
Changed lines of the file:
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@@
 <part name="FRAME1" library="frames" library_urn="urn:adsk.eagle:library:229" deviceset="A4L-LOC" device=""/>
 <part name="IC1" library="PIC32MX110F016B-I_SO" deviceset="PIC32MX110F016B-I_SO" device=""/>
-<part name="SV1" library="con-lsta" library_urn="urn:adsk.eagle:library:161" deviceset="FE06W" device="" package3d_urn="urn:adsk.eagle:package:8198/1"/>
+<part name="ICSP" library="con-lsta" library_urn="urn:adsk.eagle:library:161" deviceset="FE06W" device="" package3d_urn="urn:adsk.eagle:package:8198/1"/>
 <part name="GND4" library="supply1" library_urn="urn:adsk.eagle:library:371" deviceset="GND" device=""/>
 <part name="GND7" library="supply1" library_urn="urn:adsk.eagle:library:371" deviceset="GND" device=""/>
@@
 <part name="C6" library="rcl" library_urn="urn:adsk.eagle:library:334" deviceset="C-EU" device="C0603K" package3d_urn="urn:adsk.eagle:package:23680/2" value="100n"/>
 <part name="GND12" library="supply1" library_urn="urn:adsk.eagle:library:371" deviceset="GND" device=""/>
-<part name="T1" library="transistor-neu-to92" library_urn="urn:adsk.eagle:library:397" deviceset="*-NPN-" device="SOT23-BEC" package3d_urn="urn:adsk.eagle:package:28748/2" technology="BC817-16"/>
+<part name="T1" library="transistor-npn" library_urn="urn:adsk.eagle:library:398" deviceset="BC817*" device="SMD" package3d_urn="urn:adsk.eagle:package:28990/2" technology="-16LT1"/>
 <part name="R4" library="resistor" library_urn="urn:adsk.eagle:library:348" deviceset="R-US_" device="M0805" package3d_urn="urn:adsk.eagle:package:26079/1" value="100k"/>
 <part name="R3" library="resistor" library_urn="urn:adsk.eagle:library:348" deviceset="R-US_" device="M0805" package3d_urn="urn:adsk.eagle:package:26079/1" value="10k"/>
@@
 <instance part="FRAME1" gate="G$1" x="0" y="0"/>
 <instance part="IC1" gate="G$1" x="63.5" y="104.14"/>
-<instance part="SV1" gate="G$1" x="15.24" y="160.02" rot="MR180"/>
+<instance part="ICSP" gate="G$1" x="15.24" y="160.02" rot="MR180"/>
 <instance part="GND4" gate="1" x="60.96" y="58.42"/>
 <instance part="GND7" gate="1" x="190.5" y="58.42"/>
@@
 </segment>
 <segment>
-<pinref part="SV1" gate="G$1" pin="3"/>
+<pinref part="ICSP" gate="G$1" pin="3"/>
 <wire x1="22.86" y1="160.02" x2="25.4" y2="160.02" width="0.1524" layer="91"/>
 <wire x1="25.4" y1="160.02" x2="25.4" y2="149.86" width="0.1524" layer="91"/>
@@
 </segment>
 <segment>
-<pinref part="SV1" gate="G$1" pin="2"/>
+<pinref part="ICSP" gate="G$1" pin="2"/>
 <wire x1="22.86" y1="162.56" x2="43.18" y2="162.56" width="0.1524" layer="91"/>
 <pinref part="+3V33" gate="G$1" pin="+3V3"/>
@@
 <wire x1="60.96" y1="124.46" x2="55.88" y2="124.46" width="0.1524" layer="91"/>
 <pinref part="R2" gate="G$1" pin="2"/>
-<pinref part="SV1" gate="G$1" pin="1"/>
+<pinref part="ICSP" gate="G$1" pin="1"/>
 <wire x1="22.86" y1="165.1" x2="60.96" y2="165.1" width="0.1524" layer="91"/>
 <wire x1="60.96" y1="165.1" x2="60.96" y2="124.46" width="0.1524" layer="91"/>
@@
 </segment>
 <segment>
-<pinref part="SV1" gate="G$1" pin="5"/>
+<pinref part="ICSP" gate="G$1" pin="5"/>
 <wire x1="22.86" y1="154.94" x2="38.1" y2="154.94" width="0.1524" layer="91"/>
 <wire x1="38.1" y1="154.94" x2="38.1" y2="152.4" width="0.1524" layer="91"/>
@@
 </segment>
 <segment>
-<pinref part="SV1" gate="G$1" pin="4"/>
+<pinref part="ICSP" gate="G$1" pin="4"/>
 <wire x1="22.86" y1="157.48" x2="40.64" y2="157.48" width="0.1524" layer="91"/>
 <label x="40.64" y="157.48" size="1.778" layer="95" xref="yes"/>

Commit message: laser sensor gerber updated
Parts:
- added JMP1, JMP2, JMP3, JMP4: 0R-JUMPA, jump-0r-smd:0R-JUMPA
- added Q3, Q4: BC817, transistor-npn:BC817-16LT1SMD
- added R12, R20, R21, R25: 10k, rcl:R-US_R0805
- added R18, R23: 100k, rcl:R-US_R0805
- ICSP: device con-lsta:FE06W -> con-lsta:FE06-1
- J6: SPICEPREFIX (none) -> E
- J7: SPICEPREFIX (none) -> B
- LED9: SPICEPREFIX (none) -> L
- Q2: SPICEPREFIX (none) -> Q
- TP37: SPICEPREFIX (none) -> X
Connections:
- new net N$11: J6.4, JMP4-0R.2
- new net N$13: Q4.B, R21.2, R23.1
- new net N$16: J7.2, JMP2-0R.2, LED9.A
- new net N$21: J4.4, JMP3-0R.2
- new net N$26: Q3.B, R12.2, R18.1
- new net N$27: J4.2, R12.1
- new net N$28: J6.2, R21.1
- new net N$6: J5.2, JMP1-0R.2, LED8.A
- net +3V3: now also JMP1-0R.1, JMP2-0R.1, JMP3-0R.1, JMP4-0R.1, R20.2, R25.2; no longer J4.4, J6.4
- net +5V: now also JMP1-0R.3, JMP2-0R.3, JMP3-0R.3, JMP4-0R.3; no longer J5.2, J7.2, LED8.A, LED9.A
- net GND: now also Q3.E, Q4.E, R18.2, R23.2
- net INT_LEFT: now also Q4.C, R25.1; no longer J6.2
- net INT_RIGHT: now also Q3.C, R20.1; no longer J4.2
Other:
- moved on the sheet: J4, J5, J6, J7, LED8, LED9, Q1, Q2, R38, R39, R40, R41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

Commit message: TPS6300x inductors changed
Parts:
- C17, C18, C19, C20, C21: device rcl:C-EUC0805K -> rcl:C-EUC0402K
- L1, L2, L3: device LQM21PN2R2MC0D:LQM21PN2R2MC0D -> 0402_inductor:INDUCTOR
- L4, L5: device VLF4012AT-3R3M1R3:VLF4012AT-3R3M1R3 -> LPS3015-222MRB:LPS3015-222MRB
- R1, R2, R3, R4, R5: device resistor:R-US_M0805 -> rcl:R-US_R0805
- R14: value 560 -> 620
- R36: RS_PART_NUMBER (none) -> 740-8978
- R37: device rcl:R-US_M0805 -> rcl:R-US_R0805; RS_PART_NUMBER (none) -> 740-8978
Connections:
- net N$32: now also L1.P$1, L2.P$1; no longer L1.1, L2.1
- net N$33: now also L1.P$2, L3.P$1; no longer L1.2, L3.1
- net N$35: now also L3.P$2; no longer L3.2
- net N$36: now also L2.P$2; no longer L2.2

Commit message: Version added
Other:
- note added: "v0.1_α"
Changed lines of the file:
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@@
 <?xml version="1.0" encoding="utf-8"?>
 <!DOCTYPE eagle SYSTEM "eagle.dtd">
-<eagle version="9.1.0">
+<eagle version="9.1.3">
 <drawing>
 <settings>
@@
 1: Application
 0: Bootloader</text>
+<text x="246.38" y="5.08" size="2.54" layer="94">v0.1_α</text>
 </plain>
 <instances>
@@
 <description>USB to UART bridge</description>
 <plain>
+<text x="246.38" y="5.08" size="2.54" layer="94">v0.1_α</text>
 </plain>
 <instances>
@@
 <text x="20.32" y="10.16" size="1.778" layer="91">Short SJ1 to use the +3v3
 provided by the debugger</text>
+<text x="246.38" y="5.08" size="2.54" layer="94">v0.1_α</text>
 </plain>
 <instances>
@@
 <plain>
 <text x="111.76" y="53.34" size="1.778" layer="91">I2C address: 0100000x</text>
+<text x="246.38" y="5.08" size="2.54" layer="94">v0.1_α</text>
 </plain>
 <instances>
@@
 DO NOT MOUNT R23</text>
 <text x="124.46" y="147.32" size="1.778" layer="91">CHG LED exposed to user</text>
+<text x="246.38" y="5.08" size="2.54" layer="94">v0.1_α</text>
 </plain>
 <instances>
@@
 <text x="132.08" y="63.5" size="1.778" layer="91">TEST NEEDED
 ON R33</text>
+<text x="246.38" y="5.08" size="2.54" layer="94">v0.1_α</text>
 </plain>
 <instances>
@@
 <plain>
 <text x="116.84" y="63.5" size="1.778" layer="91">I2C address: 1010000x</text>
+<text x="246.38" y="5.08" size="2.54" layer="94">v0.1_α</text>
 </plain>
 <instances>
@@
 <description>Voltage regulators</description>
 <plain>
+<text x="246.38" y="5.08" size="2.54" layer="94">v0.1_α</text>
 </plain>
 <instances>
@@
 <text x="137.16" y="124.46" size="1.778" layer="91">TEST THIS SITUTATION
 CAREFULLY</text>
+<text x="246.38" y="5.08" size="2.54" layer="94">v0.1_α</text>
 </plain>
 <instances>

Commit message: Added revision info. PDF updated
Other:
- note added: "Zampieri Gabriele Speed'o'Meter v 0.1-alpha https://github.com/gabbla/speedometer"
- note removed: "TEST THIS SITUTATION CAREFULLY"
- note removed: "v0.1_α"
Changed lines of the file:
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@@
 <drawing>
 <settings>
-<setting alwaysvectorfont="yes"/>
+<setting alwaysvectorfont="no"/>
 <setting verticaltext="up"/>
 </settings>
-<grid distance="0.1" unitdist="inch" unit="inch" style="lines" multiple="1" display="yes" altdistance="0.01" altunitdist="inch" altunit="inch"/>
+<grid distance="0.05" unitdist="inch" unit="inch" style="lines" multiple="1" display="no" altdistance="0.01" altunitdist="inch" altunit="inch"/>
 <layers>
 <layer number="1" name="Top" color="4" fill="1" visible="no" active="no"/>
@@
 1: Application
 0: Bootloader</text>
-<text x="246.38" y="5.08" size="2.54" layer="94">v0.1_α</text>
+<text x="163.83" y="7.62" size="2.032" layer="94">Zampieri Gabriele
+Speed'o'Meter
+v 0.1-alpha
+https://github.com/gabbla/speedometer</text>
 </plain>
 <instances>
@@
 <description>USB to UART bridge</description>
 <plain>
-<text x="246.38" y="5.08" size="2.54" layer="94">v0.1_α</text>
+<text x="163.83" y="7.62" size="2.032" layer="94">Zampieri Gabriele
+Speed'o'Meter
+v 0.1-alpha
+https://github.com/gabbla/speedometer</text>
 </plain>
 <instances>
@@
 <text x="20.32" y="10.16" size="1.778" layer="91">Short SJ1 to use the +3v3
 provided by the debugger</text>
-<text x="246.38" y="5.08" size="2.54" layer="94">v0.1_α</text>
+<text x="163.83" y="7.62" size="2.032" layer="94">Zampieri Gabriele
+Speed'o'Meter
+v 0.1-alpha
+https://github.com/gabbla/speedometer</text>
 </plain>
 <instances>
@@
 <plain>
 <text x="111.76" y="53.34" size="1.778" layer="91">I2C address: 0100000x</text>
-<text x="246.38" y="5.08" size="2.54" layer="94">v0.1_α</text>
+<text x="163.83" y="7.62" size="2.032" layer="94">Zampieri Gabriele
+Speed'o'Meter
+v 0.1-alpha
+https://github.com/gabbla/speedometer</text>
 </plain>
 <instances>
@@
 DO NOT MOUNT R23</text>
 <text x="124.46" y="147.32" size="1.778" layer="91">CHG LED exposed to user</text>
-<text x="246.38" y="5.08" size="2.54" layer="94">v0.1_α</text>
+<text x="163.83" y="7.62" size="2.032" layer="94">Zampieri Gabriele
+Speed'o'Meter
+v 0.1-alpha
+https://github.com/gabbla/speedometer</text>
 </plain>
 <instances>
@@
 <text x="132.08" y="63.5" size="1.778" layer="91">TEST NEEDED
 ON R33</text>
-<text x="246.38" y="5.08" size="2.54" layer="94">v0.1_α</text>
+<text x="163.83" y="7.62" size="2.032" layer="94">Zampieri Gabriele
+Speed'o'Meter
+v 0.1-alpha
+https://github.com/gabbla/speedometer</text>
 </plain>
 <instances>
@@
 <plain>
 <text x="116.84" y="63.5" size="1.778" layer="91">I2C address: 1010000x</text>
-<text x="246.38" y="5.08" size="2.54" layer="94">v0.1_α</text>
+<text x="163.83" y="7.62" size="2.032" layer="94">Zampieri Gabriele
+Speed'o'Meter
+v 0.1-alpha
+https://github.com/gabbla/speedometer</text>
 </plain>
 <instances>
@@
 <description>Voltage regulators</description>
 <plain>
-<text x="246.38" y="5.08" size="2.54" layer="94">v0.1_α</text>
+<text x="163.83" y="7.62" size="2.032" layer="94">Zampieri Gabriele
+Speed'o'Meter
+v 0.1-alpha
+https://github.com/gabbla/speedometer</text>
 </plain>
 <instances>
@@
 <description>Sensing</description>
 <plain>
-<text x="12.7" y="124.46" size="1.778" layer="91">TEST THIS SITUTATION
-CAREFULLY</text>
-<text x="137.16" y="124.46" size="1.778" layer="91">TEST THIS SITUTATION
-CAREFULLY</text>
-<text x="246.38" y="5.08" size="2.54" layer="94">v0.1_α</text>
+<text x="163.83" y="7.62" size="2.032" layer="94">Zampieri Gabriele
+Speed'o'Meter
+v 0.1-alpha
+https://github.com/gabbla/speedometer</text>
 </plain>
 <instances>
