File: hardware/speedometer/speedometer.sch (EAGLE design)
At the start: 149 parts, among them IC1 PIC32MX110F016B-I_SO, IC10 24LC024SN, IC11 MAX16054AZT+T, IC12 TPS63001DRCT, IC13 TPS63002DRCT, IC2 CSTCE8M00G55-R0, IC3 CSTCE12M0G15L99-R0, IC4 MCP2200-I_SO, IC6 PCF8574T, IC7 BQ24075RGTT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

Commit message: Fixed diode (#8) and battery polarity (#5)
Parts:
- removed D1: BAT54, diode:BAT54
Connections:
- removed net N$45: D1.C, R1.2
- net +3V3: now also R1.2; no longer D1.A
- net GND: now also J2.1; no longer J2.2
- net N$10: now also J2.2; no longer J2.1
Other:
- moved on the sheet: J2
Changed lines of the file:
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@@
 <setting verticaltext="up"/>
 </settings>
-<grid distance="0.05" unitdist="inch" unit="inch" style="lines" multiple="1" display="no" altdistance="0.01" altunitdist="inch" altunit="inch"/>
+<grid distance="0.1" unitdist="inch" unit="inch" style="lines" multiple="1" display="yes" altdistance="0.01" altunitdist="inch" altunit="inch"/>
 <layers>
 <layer number="1" name="Top" color="4" fill="1" visible="no" active="no"/>
@@
 <part name="GND2" library="supply1" library_urn="urn:adsk.eagle:library:371" deviceset="GND" device=""/>
 <part name="+3V33" library="supply1" library_urn="urn:adsk.eagle:library:371" deviceset="+3V3" device=""/>
-<part name="D1" library="diode" library_urn="urn:adsk.eagle:library:210" deviceset="BAT54" device="" package3d_urn="urn:adsk.eagle:package:43389/2"/>
 <part name="FRAME2" library="frames" library_urn="urn:adsk.eagle:library:229" deviceset="A4L-LOC" device=""/>
 <part name="IC4" library="MCP2200-I_SO" deviceset="MCP2200-I_SO" device=""/>
@@
 <instance part="R1" gate="G$1" x="40.64" y="132.08" rot="R90"/>
 <instance part="C2" gate="G$1" x="40.64" y="119.38"/>
-<instance part="+3V32" gate="G$1" x="17.78" y="139.7" rot="R90"/>
+<instance part="+3V32" gate="G$1" x="40.64" y="142.24"/>
 <instance part="GND3" gate="1" x="40.64" y="109.22"/>
 <instance part="C4" gate="G$1" x="238.76" y="78.74">
@@
 <instance part="GND2" gate="1" x="25.4" y="147.32"/>
 <instance part="+3V33" gate="G$1" x="45.72" y="162.56" rot="R270"/>
-<instance part="D1" gate="G$1" x="30.48" y="139.7"/>
 <instance part="T1" gate="G$1" x="88.9" y="25.4"/>
 <instance part="R4" gate="G$1" x="83.82" y="17.78"/>
@@
 </segment>
 <segment>
-<pinref part="+3V32" gate="G$1" pin="+3V3"/>
-<pinref part="D1" gate="G$1" pin="A"/>
-<wire x1="20.32" y1="139.7" x2="27.94" y2="139.7" width="0.1524" layer="91"/>
-</segment>
-<segment>
 <pinref part="R5" gate="G$1" pin="2"/>
 <wire x1="91.44" y1="45.72" x2="91.44" y2="48.26" width="0.1524" layer="91"/>
 <pinref part="+3V34" gate="G$1" pin="+3V3"/>
+</segment>
+<segment>
+<pinref part="R1" gate="G$1" pin="2"/>
+<wire x1="40.64" y1="139.7" x2="40.64" y2="137.16" width="0.1524" layer="91"/>
+<pinref part="+3V32" gate="G$1" pin="+3V3"/>
 </segment>
 </net>
@@
 <wire x1="22.86" y1="157.48" x2="40.64" y2="157.48" width="0.1524" layer="91"/>
 <label x="40.64" y="157.48" size="1.778" layer="95" xref="yes"/>
-</segment>
-</net>
-<net name="N$45" class="0">
-<segment>
-<pinref part="D1" gate="G$1" pin="C"/>
-<pinref part="R1" gate="G$1" pin="2"/>
-<wire x1="33.02" y1="139.7" x2="40.64" y2="139.7" width="0.1524" layer="91"/>
-<wire x1="40.64" y1="139.7" x2="40.64" y2="137.16" width="0.1524" layer="91"/>
 </segment>
 </net>
@@
 <instance part="VCC1" gate="G$1" x="195.58" y="99.06" rot="R270"/>
 <instance part="VDD5" gate="G$1" x="104.14" y="124.46"/>
-<instance part="J2" gate="G$1" x="55.88" y="91.44" rot="R270"/>
+<instance part="J2" gate="G$1" x="55.88" y="71.12" rot="R90"/>
 <instance part="GND31" gate="1" x="55.88" y="66.04"/>
 <instance part="C12" gate="G$1" x="93.98" y="111.76"/>
@@
 </segment>
 <segment>
-<pinref part="J2" gate="G$1" pin="2"/>
-<wire x1="55.88" y1="71.12" x2="55.88" y2="68.58" width="0.1524" layer="91"/>
-<pinref part="GND31" gate="1" pin="GND"/>
-</segment>
-<segment>
 <pinref part="C12" gate="G$1" pin="2"/>
 <pinref part="GND33" gate="1" pin="GND"/>
@@
 <pinref part="GND43" gate="1" pin="GND"/>
 <wire x1="91.44" y1="66.04" x2="91.44" y2="55.88" width="0.1524" layer="91"/>
+</segment>
+<segment>
+<pinref part="J2" gate="G$1" pin="1"/>
+<pinref part="GND31" gate="1" pin="GND"/>
+<wire x1="55.88" y1="71.12" x2="55.88" y2="68.58" width="0.1524" layer="91"/>
 </segment>
 </net>
@@
 <wire x1="78.74" y1="91.44" x2="78.74" y2="93.98" width="0.1524" layer="91"/>
 <junction x="78.74" y="93.98"/>
-<pinref part="J2" gate="G$1" pin="1"/>
 <wire x1="78.74" y1="93.98" x2="55.88" y2="93.98" width="0.1524" layer="91"/>
-<wire x1="55.88" y1="93.98" x2="55.88" y2="91.44" width="0.1524" layer="91"/>
 <pinref part="TP23" gate="G$1" pin="TP"/>
 <wire x1="55.88" y1="93.98" x2="55.88" y2="96.52" width="0.1524" layer="91"/>
+<pinref part="J2" gate="G$1" pin="2"/>
+<wire x1="55.88" y1="91.44" x2="55.88" y2="93.98" width="0.1524" layer="91"/>
 <junction x="55.88" y="93.98"/>
 </segment>
