File: hardware/speedometer/speedometer.sch (EAGLE design)
At the start: 124 parts, among them IC1 PIC32MX274F256DT-I_PT, IC10 TPS63001DRCT, IC11 TPS63002DRCT, IC2 CSTCE8M00G55-R0, IC3 HM-11, IC4 BQ27441DRZR-G1A, IC5 BQ24075RGTT, IC6 NRF24L01P-T, IC7 CSTCE16M0V53-R0, IC8 24LC024SN, IC9 MAX16054AZT+T, J1 10104111-0001LF, J2 BAT, J3 CONUFL001-SMD-T, J4 Right_sens, J5 Right, J6 Left_sens, J7 Left, Q1 BC817, Q2 BC817, Q3 BC817, Q4 BC817, U1 SN74AHC1G08DBVR

Commit message: wip
Parts:
- added R35: 1k5, rcl:R-US_M0805
- added STATUS: (no value), led:LED3MM
- added TP25: TPB1,27, testpad:TPB1,27
- renumbered LED2 to BT, LED3 to CHG
Connections:
- new net N$10: R35.1, STATUS.C
- net GND: now also R35.2
- net LED_STS: now also STATUS.A
- net NRF_IRQ: now also TP25.TP
Other:
- note removed: "TEST NEEDED ON R33"
Changed lines of the file:
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@@
 <setting verticaltext="up"/>
 </settings>
-<grid distance="0.1" unitdist="inch" unit="inch" style="lines" multiple="1" display="no" altdistance="0.01" altunitdist="inch" altunit="inch"/>
+<grid distance="0.1" unitdist="inch" unit="inch" style="lines" multiple="1" display="yes" altdistance="0.01" altunitdist="inch" altunit="inch"/>
 <layers>
 <layer number="1" name="Top" color="4" fill="1" visible="no" active="no"/>
@@
 <part name="C11" library="rcl" library_urn="urn:adsk.eagle:library:334" deviceset="C-EU" device="C0603K" package3d_urn="urn:adsk.eagle:package:23680/2" value="100n"/>
 <part name="GND22" library="supply1" library_urn="urn:adsk.eagle:library:371" deviceset="GND" device=""/>
-<part name="LED3" library="led" library_urn="urn:adsk.eagle:library:259" deviceset="LED" device="3MM" package3d_urn="urn:adsk.eagle:package:15797/1"/>
+<part name="CHG" library="led" library_urn="urn:adsk.eagle:library:259" deviceset="LED" device="3MM" package3d_urn="urn:adsk.eagle:package:15797/1"/>
 <part name="R16" library="rcl" library_urn="urn:adsk.eagle:library:334" deviceset="R-US_" device="R0805" package3d_urn="urn:adsk.eagle:package:23553/2" value="1k5"/>
 <part name="TP15" library="testpad" library_urn="urn:adsk.eagle:library:385" deviceset="TP" device="B1,27" package3d_urn="urn:adsk.eagle:package:27944/1" value="TPB1,27">
@@
 </part>
 <part name="R10" library="rcl" library_urn="urn:adsk.eagle:library:334" deviceset="R-US_" device="M0805" package3d_urn="urn:adsk.eagle:package:23556/1" value="470"/>
-<part name="LED2" library="led" library_urn="urn:adsk.eagle:library:259" deviceset="LED" device="3MM" package3d_urn="urn:adsk.eagle:package:15797/1"/>
+<part name="BT" library="led" library_urn="urn:adsk.eagle:library:259" deviceset="LED" device="3MM" package3d_urn="urn:adsk.eagle:package:15797/1"/>
 <part name="R9" library="rcl" library_urn="urn:adsk.eagle:library:334" deviceset="R-US_" device="M0805" package3d_urn="urn:adsk.eagle:package:23556/1" value="470"/>
 <part name="GND15" library="supply1" library_urn="urn:adsk.eagle:library:371" deviceset="GND" device=""/>
@@
 <part name="C10" library="rcl" library_urn="urn:adsk.eagle:library:334" deviceset="C-EU" device="C0805K" package3d_urn="urn:adsk.eagle:package:23681/2" value="10u"/>
 <part name="VCC1" library="supply1" library_urn="urn:adsk.eagle:library:371" deviceset="VCCINT" device=""/>
+<part name="STATUS" library="led" library_urn="urn:adsk.eagle:library:259" deviceset="LED" device="3MM" package3d_urn="urn:adsk.eagle:package:15797/1"/>
+<part name="R35" library="rcl" library_urn="urn:adsk.eagle:library:334" deviceset="R-US_" device="M0805" package3d_urn="urn:adsk.eagle:package:23556/1" value="1k5"/>
+<part name="TP25" library="testpad" library_urn="urn:adsk.eagle:library:385" deviceset="TP" device="B1,27" package3d_urn="urn:adsk.eagle:package:27944/1"/>
 </parts>
 <sheets>
@@
 <attribute name="VALUE" x="233.68" y="114.3" size="1.778" layer="96"/>
 </instance>
+<instance part="STATUS" gate="G$1" x="22.86" y="53.34" smashed="yes" rot="R90">
+<attribute name="NAME" x="27.432" y="56.896" size="1.778" layer="95" rot="R180"/>
+<attribute name="VALUE" x="27.432" y="59.055" size="1.778" layer="96" rot="R180"/>
+</instance>
+<instance part="R35" gate="G$1" x="38.1" y="53.34" smashed="yes">
+<attribute name="NAME" x="34.29" y="54.8386" size="1.778" layer="95"/>
+<attribute name="VALUE" x="34.29" y="50.038" size="1.778" layer="96"/>
+</instance>
 </instances>
 <busses>
@@
 <wire x1="45.72" y1="45.72" x2="45.72" y2="43.18" width="0.1524" layer="91"/>
 <pinref part="GND4" gate="1" pin="GND"/>
+<pinref part="R35" gate="G$1" pin="2"/>
+<wire x1="43.18" y1="53.34" x2="45.72" y2="53.34" width="0.1524" layer="91"/>
+<wire x1="45.72" y1="53.34" x2="45.72" y2="45.72" width="0.1524" layer="91"/>
+<junction x="45.72" y="45.72"/>
 </segment>
 <segment>
@@
 <label x="53.34" y="116.84" size="1.27" layer="95" font="vector" rot="R180" xref="yes"/>
 </segment>
+<segment>
+<pinref part="STATUS" gate="G$1" pin="A"/>
+<wire x1="20.32" y1="53.34" x2="15.24" y2="53.34" width="0.1524" layer="91"/>
+<label x="15.24" y="53.34" size="1.27" layer="95" font="vector" rot="R180" xref="yes"/>
+</segment>
 </net>
 <net name="N$29" class="0">
@@
 <wire x1="66.04" y1="111.76" x2="53.34" y2="111.76" width="0.1524" layer="91"/>
 <label x="53.34" y="111.76" size="1.27" layer="95" font="vector" rot="R180" xref="yes"/>
+</segment>
+</net>
+<net name="N$10" class="0">
+<segment>
+<pinref part="STATUS" gate="G$1" pin="C"/>
+<pinref part="R35" gate="G$1" pin="1"/>
+<wire x1="27.94" y1="53.34" x2="33.02" y2="53.34" width="0.1524" layer="91"/>
 </segment>
 </net>
@@
 <attribute name="VALUE" x="163.83" y="90.678" size="1.778" layer="96"/>
 </instance>
-<instance part="LED2" gate="G$1" x="175.26" y="83.82" smashed="yes" rot="R90">
+<instance part="BT" gate="G$1" x="175.26" y="83.82" smashed="yes" rot="R90">
 <attribute name="NAME" x="179.832" y="87.376" size="1.778" layer="95" rot="R180"/>
 <attribute name="VALUE" x="179.832" y="89.535" size="1.778" layer="96" rot="R180"/>
@@
 </segment>
 <segment>
-<pinref part="LED2" gate="G$1" pin="C"/>
+<pinref part="BT" gate="G$1" pin="C"/>
 <wire x1="180.34" y1="83.82" x2="185.42" y2="83.82" width="0.1524" layer="91"/>
 <pinref part="GND15" gate="1" pin="GND"/>
@@
 <segment>
 <pinref part="R9" gate="G$1" pin="2"/>
-<pinref part="LED2" gate="G$1" pin="A"/>
+<pinref part="BT" gate="G$1" pin="A"/>
 <wire x1="167.64" y1="83.82" x2="172.72" y2="83.82" width="0.1524" layer="91"/>
 </segment>
@@
 <attribute name="VALUE" x="139.7" y="101.6" size="1.778" layer="96"/>
 </instance>
-<instance part="LED3" gate="G$1" x="190.5" y="121.92" smashed="yes" rot="R270">
+<instance part="CHG" gate="G$1" x="190.5" y="121.92" smashed="yes" rot="R270">
 <attribute name="NAME" x="185.928" y="118.364" size="1.778" layer="95"/>
 <attribute name="VALUE" x="185.928" y="116.205" size="1.778" layer="96"/>
@@
 <pinref part="IC5" gate="G$1" pin="!CHG"/>
 <wire x1="180.34" y1="121.92" x2="180.34" y2="109.22" width="0.1524" layer="91"/>
-<pinref part="LED3" gate="G$1" pin="C"/>
+<pinref part="CHG" gate="G$1" pin="C"/>
 <wire x1="185.42" y1="121.92" x2="180.34" y2="121.92" width="0.1524" layer="91"/>
 <pinref part="TP17" gate="G$1" pin="TP"/>
@@
 <net name="N$12" class="0">
 <segment>
-<pinref part="LED3" gate="G$1" pin="A"/>
+<pinref part="CHG" gate="G$1" pin="A"/>
 <pinref part="R16" gate="G$1" pin="2"/>
 <wire x1="193.04" y1="121.92" x2="198.12" y2="121.92" width="0.1524" layer="91"/>
@@
 <description>nRF24L01+</description>
 <plain>
-<text x="132.08" y="63.5" size="1.778" layer="91">TEST NEEDED
-ON R33</text>
 <text x="163.83" y="7.62" size="2.032" layer="94">Zampieri Gabriele
 Speed'o'Meter
@@
 <instance part="GND32" gate="1" x="116.84" y="137.16" smashed="yes">
 <attribute name="VALUE" x="114.3" y="134.62" size="1.778" layer="96"/>
+</instance>
+<instance part="TP25" gate="G$1" x="144.78" y="76.2" smashed="yes">
+<attribute name="NAME" x="143.51" y="77.47" size="1.778" layer="95"/>
+<attribute name="TP_SIGNAL_NAME" x="146.05" y="74.93" size="1.778" layer="97"/>
 </instance>
 </instances>
@@
 <junction x="134.62" y="71.12"/>
 <label x="116.84" y="71.12" size="1.27" layer="95" font="vector" rot="R180" xref="yes"/>
-</segment>
-</net>
+<wire x1="139.7" y1="71.12" x2="144.78" y2="71.12" width="0.1524" layer="91"/>
+<junction x="139.7" y="71.12"/>
+<pinref part="TP25" gate="G$1" pin="TP"/>
+<wire x1="144.78" y1="71.12" x2="144.78" y2="73.66" width="0.1524" layer="91"/>
+</segment>
+</net>

Commit message: wip
Parts:
- removed LED5: (no value), led:LEDCHIPLED_1206
- removed TP25: TPB1,27, testpad:TPB1,27
- added C29: 1n, rcl:C-EUC0603K
- added LED2: (no value), led:LEDCHIPLED_1206
- added U2: SN74AHC1G08DBVR, SN74AHC1G08DBVR:SN74AHC1G08DBVR
- C1, C2, C4, C5, C6, C7: device rcl:C-EUC0603 -> rcl:C-EUC0603K
- C10, C13, C14, C21, C22, C25, C26, C27, C28, C3, C8, C9: device rcl:C-EUC0805K -> rcl:C-EUC0603K
- J7: SPICEPREFIX B -> (none)
- Q3: SPICEPREFIX Q -> (none)
- R1, R10, R2, R3, R35, R4, R5, R6, R7, R8, R9: device rcl:R-US_M0805 -> rcl:R-US_R0603
- R12, R13, R14, R15, R16, R17, R18, R19, R20, R21, R22, R23, R24, R25, R26, R27, R28, R29, R30, R31, R32, R33, R34: device rcl:R-US_R0805 -> rcl:R-US_R0603
- TP24: SPICEPREFIX X -> (none); TP_SIGNAL_NAME TP_L_SX -> TP_L_DX
Connections:
- removed net INT_LEFT: Q4.C, R34.1
- removed net INT_RIGHT: Q1.C, R26.1
- removed net LASER_LEFT_CTL: R29.1
- removed net LEFT_STS: J6.3
- removed net N$20: LED5.C, R32.2
- removed net RIGHT_STS: J4.3
- new net N$15: LED2.C, R32.2
- new net N$16: R29.1, U2.Y
- net +3V3: now also C29.1, U2.VCC
- net +5V: now also LED2.A; no longer LED5.A
- net CTL_L: now also U2.B
- net GND: now also C29.2, U2.GND
- net IN_L: now also Q4.C, R34.1
- net IN_R: now also Q1.C, R26.1
- net LASER_MOD: now also U2.A
- net NRF_IRQ: no longer TP25.TP
- net STS_L: now also J6.3
- net STS_R: now also J4.3
Other:
- moved on the sheet: J7, Q3, R29, R30, R32, TP24
