File: hardware/speedometer/speedometer.brd (EAGLE design)
At the start: 69.8 x 54.6 mm, 127 parts, among them IC1 PIC32MX274F256DT-I_PT, IC10 TPS63001DRCT, IC11 TPS63002DRCT, IC2 CSTCE8M00G55-R0, IC3 HM-11, IC4 BQ27441DRZR-G1A, IC5 BQ24075RGTT, IC6 NRF24L01P-T, IC7 CSTCE16M0V53-R0, IC8 24LC024SN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

Commit message: wip
Parts:
- removed LED5: (no value), led:CHIPLED_1206
- removed TP25: TPB1,27, testpad:B1,27
- added C29: 1n, rcl:C0603K
- added LED2: (no value), led:CHIPLED_1206
- added U2: SN74AHC1G08DBVR, SN74AHC1G08DBVR:SOT95P280X145-5N
- C1, C2, C4, C5, C6, C7: device rcl:C0603 -> rcl:C0603K
- C10, C13, C14, C21, C22, C25, C26, C27, C28, C3, C8, C9: device rcl:C0805K -> rcl:C0603K
- R1, R10, R2, R3, R35, R4, R5, R6, R7, R8, R9: device rcl:M0805 -> rcl:R0603
- R12, R13, R14, R15, R16, R17, R18, R19, R20, R21, R22, R23, R24, R25, R26, R27, R28, R29, R30, R31, R32, R33, R34: device rcl:R0805 -> rcl:R0603
- moved TP17 165.0 mm to (61.0, 16.5)
- moved TP14 156.1 mm to (61.0, 18.0)
- moved TP13 153.6 mm to (67.0, 26.0)
- moved LED4 144.2 mm to (65.4, 37.8), turned to 270 degrees
- moved C1 122.8 mm to (39.8, 25.4)
- moved C2 118.5 mm to (32.2, 34.4), turned to 90 degrees
- moved C4 118.4 mm to (22.0, 24.6), turned to 180 degrees
- moved TP8 112.4 mm to (38.2, 37.2)
- moved TP23 106.2 mm to (50.0, 50.7)
- moved IC8 101.2 mm to (29.2, 39.4), turned to 270 degrees
- moved TP10 99.4 mm to (6.40, 7.20)
- moved TP7 98.7 mm to (40.8, 35.0)
- moved R33 95.7 mm to (16.2, 40.8), turned to 270 degrees
- moved TP9 93.5 mm to (6.40, 9.60)
- moved R28 93.3 mm to (65.4, 35.8)
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Connections:
- removed net INT_LEFT: Q4.C, R34.1
- removed net INT_RIGHT: Q1.C, R26.1
- removed net LASER_LEFT_CTL: R29.1
- removed net LEFT_STS: J6.3
- removed net N$20: LED5.C, R32.2
- removed net RIGHT_STS: J4.3
- new net N$15: LED2.C, R32.2
- new net N$16: R29.1, U2.4
- net +3V3: now also C29.1, U2.5
- net +5V: now also LED2.A; no longer LED5.A
- net CTL_L: now also U2.2
- net GND: now also C29.2, U2.3
- net IN_L: now also Q4.C, R34.1
- net IN_R: now also Q1.C, R26.1
- net LASER_MOD: now also U2.1
- net NRF_IRQ: no longer TP25.TP
- net STS_L: now also J6.3
- net STS_R: now also J4.3
Routing:
- net I2C2_SCL: track 0.00 -> 49.2 mm, vias 0 -> 2
- net I2C2_SDA: track 0.00 -> 43.5 mm, vias 0 -> 2
- net +5V: track 0.00 -> 30.9 mm
- net SYS_EN: track 29.4 -> 0.00 mm, vias 3 -> 0
- net +3V3: track 0.00 -> 24.7 mm, vias 0 -> 1
- net N$4: track 0.00 -> 23.2 mm, vias 0 -> 2
- net U1_RX: track 24.0 -> 5.27 mm
- net !MCLR: track 17.7 -> 0.00 mm
- net N$1: track 0.00 -> 17.0 mm
- net PGED: track 10.9 -> 0.00 mm
- net N$38: track 0.00 -> 10.3 mm
- net BQ_1V8: track 3.24 -> 13.4 mm
- net PGEC: track 9.01 -> 0.00 mm
- net N$3: track 0.00 -> 8.42 mm
- net NRF_IRQ: track 16.5 -> 24.2 mm
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- added copper zone on layer 1, net VDD
- removed copper zone on layer 1, net N$34
- removed copper zone on layer 1, net N$5
- removed copper zone on layer 1, net N$59
- removed copper zone on layer 1, net N$61

Commit message: wip, mostly done
Parts:
- removed JP1, JP2: (no value), pinhead:1X02
- added X1, X2: TSW-102-07-G-S, con-samtec:TSW-102-XX-G-S
- SV1: device con-lsta:FE06 -> con-lstb:MA03-2
- moved TP15 137.8 mm to (36.2, 4.60)
- moved R6 126.1 mm to (35.4, 33.2)
- moved TP18 123.5 mm to (15.2, 8.75)
- moved R5 120.2 mm to (35.0, 35.6), turned to 180 degrees
- moved R25 119.8 mm to (53.8, 49.2), turned to 90 degrees
- moved TP22 116.7 mm to (58.8, 30.8)
- moved TP20 115.7 mm to (48.4, 3.00)
- moved TP21 113.3 mm to (48.2, 23.5), turned to 0 degrees
- moved R19 109.8 mm to (35.0, 44.0), turned to 180 degrees
- moved SV1 96.4 mm to (42.2, 19.4), turned to 0 degrees
- moved R8 93.7 mm to (15.0, 29.0), turned to 270 degrees
- moved R26 93.2 mm to (50.2, 45.8)
- moved C15 90.4 mm to (37.5, 39.5), turned to 270 degrees
- moved TP19 90.3 mm to (48.2, 26.0)
- moved TP16 89.3 mm to (27.2, 14.6)
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Connections:
- net +3V3: now also X2.1; no longer JP2.1
- net BL_TRIG: now also X2.2; no longer JP2.2
- net GND: now also X1.2; no longer JP1.2
- net N$41: now also X1.1; no longer JP1.1
Routing:
- net LASER_MOD: track 0.00 -> 65.6 mm, vias 0 -> 3
- net GAUGE_GP: track 4.54 -> 54.8 mm, vias 0 -> 2
- net BQ_PGOOD: track 0.00 -> 44.6 mm, vias 0 -> 4
- net SYS_EN: track 0.00 -> 42.7 mm, vias 0 -> 3
- net STS_R: track 0.00 -> 41.9 mm, vias 0 -> 1
- net IN_R: track 0.00 -> 38.4 mm, vias 0 -> 2
- net STS_L: track 0.00 -> 38.4 mm, vias 0 -> 1
- net +5V: track 30.9 -> 68.6 mm, vias 0 -> 1
- net CTL_R: track 0.00 -> 33.0 mm, vias 0 -> 2
- net U1_RX: track 5.27 -> 37.3 mm, vias 0 -> 2
- net VDD: track 23.6 -> 55.3 mm, vias 2 -> 3
- net USB_ID: track 2.75 -> 32.4 mm, vias 0 -> 2
- net N$58: track 0.00 -> 25.8 mm
- net LED_STS: track 0.00 -> 23.6 mm, vias 0 -> 1
- net U1_TX: track 10.5 -> 33.7 mm
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
Commit message: new board 4layer
Parts:
- moved CHG 154.5 mm to (-76.2, 72.4)
- moved R13 154.5 mm to (-91.4, 61.0), turned to 0 degrees
- moved J5 154.2 mm to (-88.9, 54.6), turned to 0 degrees
- moved J2 152.7 mm to (-88.9, 27.9), flipped to the top, turned to 0 degrees
- moved TP17 150.6 mm to (-74.9, 81.3)
- moved R12 149.0 mm to (-86.4, 61.0)
- moved TP19 146.6 mm to (-87.6, 81.3)
- moved C26 146.6 mm to (-88.9, 77.5)
- moved C25 145.8 mm to (-85.1, 77.5)
- moved C10 145.4 mm to (-66.0, 77.5), turned to 0 degrees
- moved C21 141.7 mm to (-77.5, 77.5)
- moved C22 141.4 mm to (-81.3, 77.5)
- moved IC5 138.1 mm to (-77.5, 24.1), turned to 0 degrees
- moved TP8 137.5 mm to (-90.2, 86.4)
- moved C1 137.0 mm to (-88.9, 72.4)
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Routing:
- net +5V: track 68.6 -> 0.00 mm, vias 1 -> 0
- net LASER_MOD: track 65.6 -> 0.00 mm, vias 3 -> 0
- net VDD: track 55.3 -> 0.00 mm, vias 3 -> 0
- net GAUGE_GP: track 54.8 -> 0.00 mm, vias 2 -> 0
- net I2C2_SCL: track 49.2 -> 0.00 mm, vias 2 -> 0
- net VCCINT: track 47.4 -> 0.00 mm, vias 2 -> 0
- net BQ_PGOOD: track 44.6 -> 0.00 mm, vias 4 -> 0
- net I2C2_SDA: track 44.4 -> 0.00 mm, vias 2 -> 0
- net SYS_EN: track 42.7 -> 0.00 mm, vias 3 -> 0
- net STS_R: track 41.9 -> 0.00 mm, vias 1 -> 0
- net IN_R: track 38.4 -> 0.00 mm, vias 2 -> 0
- net STS_L: track 38.4 -> 0.00 mm, vias 1 -> 0
- net U1_RX: track 37.3 -> 0.00 mm, vias 2 -> 0
- net U1_TX: track 33.7 -> 0.00 mm
- net CTL_R: track 33.0 -> 0.00 mm, vias 2 -> 0
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- removed copper zone on layer 1, net +3V3
- removed copper zone on layer 1, net +5V
- removed copper zone on layer 1, net VBAT
- removed copper zone on layer 1, net VCCINT
- removed copper zone on layer 1, net VDD
Other:
- board size 69.8 x 54.6 mm -> 160 x 100 mm

Commit message: new outline size
Other:
- board size 160 x 100 mm -> 70 x 55 mm
Changed lines of the file:
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@@
 <setting verticaltext="up"/>
 </settings>
-<grid distance="50" unitdist="mil" unit="mil" style="lines" multiple="1" display="no" altdistance="5" altunitdist="mil" altunit="mil"/>
+<grid distance="50" unitdist="mil" unit="mm" style="lines" multiple="1" display="yes" altdistance="5" altunitdist="mil" altunit="mil"/>
 <layers>
 <layer number="1" name="Top" color="4" fill="1" visible="yes" active="yes"/>
@@
 <board>
 <plain>
-<wire x1="0" y1="0" x2="160" y2="0" width="0" layer="20"/>
-<wire x1="160" y1="0" x2="160" y2="100" width="0" layer="20"/>
-<wire x1="160" y1="100" x2="0" y2="100" width="0" layer="20"/>
-<wire x1="0" y1="100" x2="0" y2="0" width="0" layer="20"/>
+<wire x1="0" y1="0" x2="70" y2="0" width="0" layer="20"/>
+<wire x1="70" y1="0" x2="70" y2="55" width="0" layer="20"/>
+<wire x1="70" y1="55" x2="0" y2="55" width="0" layer="20"/>
+<wire x1="0" y1="55" x2="0" y2="0" width="0" layer="20"/>
 </plain>
 <attributes>

Commit message: new size 68x55
Other:
- board size 70 x 55 mm -> 68 x 55 mm
Changed lines of the file:
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@@
 <board>
 <plain>
-<wire x1="0" y1="0" x2="70" y2="0" width="0" layer="20"/>
-<wire x1="70" y1="0" x2="70" y2="55" width="0" layer="20"/>
-<wire x1="70" y1="55" x2="0" y2="55" width="0" layer="20"/>
+<wire x1="0" y1="0" x2="68" y2="0" width="0" layer="20"/>
+<wire x1="68" y1="0" x2="68" y2="55" width="0" layer="20"/>
+<wire x1="68" y1="55" x2="0" y2="55" width="0" layer="20"/>
 <wire x1="0" y1="55" x2="0" y2="0" width="0" layer="20"/>
 </plain>

Commit message: power added
Parts:
- C10, C21, C22, C25, C26, C27, C28: device rcl:C0603K -> rcl:C0805K
- C11: value 100n -> 10u; device rcl:C0603K -> rcl:C0805K
- C12: value 4u7 -> 10u; device rcl:SMC_A -> rcl:C0805K
- moved C22 158.9 mm to (62.5, 9.75), turned to 90 degrees
- moved C26 155.7 mm to (51.2, 9.75), turned to 90 degrees
- moved J5 154.2 mm to (65.0, 45.0), turned to 270 degrees
- moved CHG 153.5 mm to (56.5, -4.75)
- moved J2 150.3 mm to (61.2, 35.2), flipped to the bottom, turned to 270 degrees
- moved R13 148.5 mm to (55.0, 36.4), turned to 90 degrees
- moved C21 145.5 mm to (55.8, 19.0), turned to 90 degrees
- moved R12 145.4 mm to (57.0, 36.4), turned to 270 degrees
- moved C25 145.4 mm to (48.0, 19.0), turned to 90 degrees
- moved L4 138.6 mm to (52.0, 14.8), turned to 180 degrees
- moved R17 138.2 mm to (65.0, 18.0), turned to 180 degrees
- moved IC5 137.5 mm to (60.0, 23.0), turned to 270 degrees
- moved C10 135.1 mm to (59.0, 26.2), turned to 180 degrees
- moved C24 135.0 mm to (57.0, 14.2), turned to 180 degrees
- moved C11 125.4 mm to (65.0, 21.0)
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Connections:
- net BQ_1V8: no longer R12.1
- net GND: now also C12.2, IC10.P$1, IC10.P$2, IC10.P$3, IC10.P$4, IC11.P$1, IC11.P$2, IC11.P$3, IC11.P$4, R12.1; no longer C12.-
- net VCCINT: now also C12.1; no longer C12.+
Routing:
- net _VBAT: track 0.00 -> 18.6 mm, vias 0 -> 5
- net VBAT: track 0.00 -> 9.27 mm
- net N$30: track 0.00 -> 5.39 mm
- net N$60: track 0.00 -> 5.13 mm
- net N$62: track 0.00 -> 4.63 mm
- net N$7: track 0.00 -> 4.17 mm
- net N$61: track 0.00 -> 3.89 mm
- net N$59: track 0.00 -> 3.89 mm
- net N$5: track 0.00 -> 3.58 mm
- net N$34: track 0.00 -> 3.58 mm
- net GAUGE_GP: track 0.00 -> 3.06 mm
- net BQ_1V8: track 0.00 -> 2.92 mm
- net N$9: track 0.00 -> 2.90 mm
- added copper zone on layer 1, net VBAT
Other:
- board text added: "GF: - Induttori TPS - Shunt batteria - Power distribution"

Commit message: wip
Parts:
- C3: device rcl:C0603K -> rcl:C0805K
- SV1: device con-lstb:MA03-2 -> con-lstb:MA06-1
- moved IC8 138.8 mm to (48.3, 38.7), turned to 90 degrees
- moved IC9 123.0 mm to (39.0, 11.4), turned to 90 degrees
- moved C1 120.3 mm to (22.4, 26.8), turned to 180 degrees
- moved IC7 117.8 mm to (53.2, 75.8)
- moved BT 116.1 mm to (10.0, 4.00)
- moved STATUS 109.3 mm to (18.0, 4.00)
- moved C20 103.5 mm to (42.8, 36.0), turned to 270 degrees
- moved IC6 92.3 mm to (42.0, 75.9)
- moved C3 87.2 mm to (32.0, 18.0), turned to 270 degrees
- moved J1 86.0 mm to (28.0, 5.00)
- moved X1 84.2 mm to (12.7, 33.7), turned to 90 degrees
- moved IC1 83.6 mm to (32.0, 27.6), turned to 90 degrees
- moved C4 80.3 mm to (41.4, 27.6)
- moved C2 78.4 mm to (35.2, 18.6), turned to 270 degrees
- moved R2 74.8 mm to (8.89, 34.9)
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Routing:
- net I2C2_SCL: track 0.00 -> 28.3 mm
- net I2C2_SDA: track 0.00 -> 27.8 mm
- net +3V3: track 0.00 -> 22.5 mm, vias 0 -> 5
- net N$41: track 0.00 -> 8.05 mm
- net N$58: track 0.00 -> 6.61 mm
- net N$19: track 0.00 -> 6.39 mm
- net N$11: track 0.00 -> 6.39 mm
- net !MCLR: track 0.00 -> 6.03 mm
- net N$21: track 0.00 -> 3.19 mm

Commit message: wip
Parts:
- added IC12: SN65220DBVRG4, SN65220DBVRG4:SOT95P280X145-6N
- IC8: value 24LC024SN -> 24LC024ST; device microchip:SO-08 -> microchip:TSSOP8
- moved TP17 152.8 mm to (55.9, 2.35)
- moved TP18 146.3 mm to (46.0, 9.05)
- moved TP8 138.5 mm to (38.5, 35.0)
- moved TP7 135.7 mm to (40.5, 35.0)
- moved U1 133.3 mm to (53.3, 42.1), turned to 90 degrees
- moved TP6 129.4 mm to (39.5, 36.8)
- moved TP5 128.4 mm to (43.5, 36.8)
- moved R35 126.6 mm to (21.9, 4.00)
- moved TP14 124.7 mm to (57.4, 29.1)
- moved TP4 123.5 mm to (42.5, 35.0)
- moved R28 123.0 mm to (58.4, 43.2), turned to 180 degrees
- moved R27 119.5 mm to (55.1, 46.1), turned to 270 degrees
- moved TP3 117.3 mm to (41.5, 36.8)
- moved TP16 116.1 mm to (28.8, 18.1)
- moved C14 115.3 mm to (37.0, 45.0), turned to 180 degrees
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Connections:
- net GND: now also IC12.2, IC12.5
- net USB_D+: now also IC12.1, IC12.6
- net USB_D-: now also IC12.3, IC12.4
Routing:
- net LASER_MOD: track 0.00 -> 70.5 mm, vias 0 -> 4
- net SYS_EN: track 0.00 -> 48.0 mm, vias 0 -> 3
- net GAUGE_GP: track 3.06 -> 50.6 mm, vias 0 -> 2
- net !MCLR: track 6.03 -> 50.9 mm, vias 0 -> 1
- net BQ_PGOOD: track 0.00 -> 43.5 mm, vias 0 -> 4
- net STS_L: track 0.00 -> 41.7 mm, vias 0 -> 1
- net STS_R: track 0.00 -> 38.4 mm, vias 0 -> 1
- net PGED: track 0.00 -> 37.3 mm, vias 0 -> 1
- net U1_RX: track 0.00 -> 36.6 mm
- net PGEC: track 0.00 -> 35.1 mm, vias 0 -> 1
- net USB_ID: track 0.00 -> 30.4 mm, vias 0 -> 2
- net LED_STS: track 0.00 -> 28.7 mm, vias 0 -> 1
- net U1_TX: track 0.00 -> 28.3 mm
- net CTL_R: track 0.00 -> 26.1 mm, vias 0 -> 2
- net !BAT_CHG: track 0.00 -> 24.9 mm, vias 0 -> 1
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